File: pcbs/Charge_Case/Charge_Case.kicad_pcb (KiCad board)
At the start: 2 copper layers, 197.5 x 33 mm, 39 parts, among them J1 GSB1C41110SSHR, J10 Conn_01x01, J11 USB4180-03-0120-C, J12 Conn_01x01, J13 Conn_01x01, J14 USB4180-03-0120-C, J15 Conn_01x01, J16 Conn_01x01, J17 USB4180-03-0120-C, J18 Conn_01x01, J19 Conn_01x01, J2 USB4180-03-0120-C, J20 USB4180-03-0120-C, J21 Conn_01x01, J22 Conn_01x01, J23 USB4180-03-0120-C, J24 Conn_01x01, J25 Conn_01x01, J26 USB4180-03-0120-C, J27 Conn_01x01, J28 Conn_01x01, J29 USB4180-03-0120-C, J3 Conn_01x01, J30 Conn_01x01, J31 Conn_01x01, J32 USB4180-03-0120-C, J33 Conn_01x01, J34 Conn_01x01, J35 USB4180-03-0120-C, J36 Conn_01x01, J37 Conn_01x01, J4 Conn_01x01, J5 USB4180-03-0120-C, J6 Conn_01x01, J7 Conn_01x01, J8 USB4180-03-0120-C, J9 Conn_01x01

Commit message: update minibot fw, add pcb ordered packages
Parts:
- added H1: MountingHole_Pad, MountingHole:MountingHole_2.7mm_M2.5_DIN965_Pad_TopOnly, F.Cu at (81.1, 100.0)
- added H2: MountingHole_Pad, MountingHole:MountingHole_2.7mm_M2.5_DIN965_Pad_TopOnly, F.Cu at (213.1, 100.0)
- added H3: MountingHole_Pad, MountingHole:MountingHole_2.7mm_M2.5_DIN965_Pad_TopOnly, F.Cu at (147.1, 100.0)
Routing:
- net GND: track 49.5 -> 69.4 mm, vias 26 -> 32
- net /CC1: track 333.1 -> 337.8 mm
- net /CC2: track 305.9 -> 310.6 mm
