File: pcbs/MiniBot_MainBoard/MiniBot.kicad_sch (KiCad schematic)
At the start: 42 parts, among them IC1 MMC5633NJL, IC2 MIC23050-SYML-TR, J1 Conn_01x08, J2 Conn_01x02, J3 GSB1C41110SSHR, U1 ESP32-C3-MINI-1-H4X, U3 MCP73832-2-OT

Commit message: fix stupid bad led symbol, general improvements to minibot fw
Connections:
- net +BATT: now also LED1.4 (R6+); no longer LED1.3 (R6+)
- net LED_R: now also LED1.3 (R6-); no longer LED1.4 (R6-)

Commit message: updoots
Parts:
- R4: value 10k -> 1k
Changed lines of the file:
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@@
       (effects (font (size 1.27 1.27)) (justify left))
     )
-    (property "Value" "10k" (at 143.51 158.75 0)
+    (property "Value" "1k" (at 143.51 158.75 0)
       (effects (font (size 1.27 1.27)) (justify left))
     )
